File: Makers-Unified-Controller/Makers-Unified-Controller.sch (KiCad schematic (older format))
At the start: 61 parts

Commit message: Completed schematic
Parts:
- removed C?: 1u, symbol Device:C
- removed J?: Battery_Connection, symbol Connector:Conn_01x02_Female
- removed J?: USB_C_Receptacle, symbol Connector:USB_C_Receptacle
- removed R? (x2): 5.1k, symbol Device:R
- removed SW?: SW_Push, symbol Switch:SW_Push
- removed U?: ESP32-WROOM-32, RF_Module:ESP32-WROOM-32, symbol RF_Module:ESP32-WROOM-32
- removed U?: MCP73811T-420I-OT, Package_TO_SOT_SMD:SOT-23-5, symbol Battery_Management:MCP73811T-420I-OT
- added BT?: BC4AAW, Footprint_Imports:BAT_BC4AAW, symbol Project_Imports:BC4AAW
- added H? (x5): MountingHole, MountingHole:MountingHole_3.2mm_M3_Pad_Via, symbol Mechanical:MountingHole
- added J?: USB_B_Micro, Footprint_Imports:AMPHENOL_10118192-0002LF, symbol Connector:USB_B_Micro
- added J?: backup_PROG, Footprint_Imports:backup_prog_header, symbol Connector:Conn_01x06_Female
- added SW?: SW_RIGHT_ANGLE, Footprint_Imports:1825027-8, symbol Switch:SW_Push
- added U?: ESP32-WROOM-32D, RF_Module:ESP32-WROOM-32, symbol RF_Module:ESP32-WROOM-32D
- A?: footprint (none) -> Footprint_Imports:SSD1306
- C? (x2): footprint (none) -> Capacitor_SMD:C_0805_2012Metric_Pad1.18x1.45mm_HandSolder; digikey_part_number (none) -> 1276-1099-1-ND
- C? (x3): footprint (none) -> Capacitor_SMD:C_0805_2012Metric_Pad1.18x1.45mm_HandSolder; digikey_part_number (none) -> 1276-6455-1-ND
- C? (x3): footprint (none) -> Capacitor_SMD:C_0805_2012Metric_Pad1.18x1.45mm_HandSolder; digikey_part_number (none) -> 1276-1275-1-ND
- D?: value D_Schottky -> CDBA340-G; footprint (none) -> Diode_SMD:D_SMA; digikey_part_number (none) -> 641-1101-1-ND
- D?: footprint (none) -> LED_SMD:LED_0805_2012Metric_Pad1.15x1.40mm_HandSolder; digikey_part_number (none) -> 160-1218-1-ND
- D?: footprint (none) -> LED_SMD:LED_0805_2012Metric_Pad1.15x1.40mm_HandSolder; digikey_part_number (none) -> 732-4982-1-ND
- L?: footprint (none) -> Footprint_Imports:NRS5024T4R7MMGJ; digikey_part_number (none) -> 587-5937-1-ND
- Q? (x2): digikey_part_number (none) -> 3757-MMBT3904_R1_00001CT-ND
- Q?: value FDN340P -> SI2305B-TP; digikey_part_number (none) -> SI2305B-TPMSCT-ND
- R? (x18): footprint (none) -> Resistor_SMD:R_0805_2012Metric_Pad1.20x1.40mm_HandSolder; digikey_part_number (none) -> RMCF0805JT10K0CT-ND
- R?: footprint (none) -> Resistor_SMD:R_0805_2012Metric_Pad1.20x1.40mm_HandSolder; digikey_part_number (none) -> RMCF0805JT47K0CT-ND
- R? (x2): footprint (none) -> Resistor_SMD:R_0805_2012Metric_Pad1.20x1.40mm_HandSolder; digikey_part_number (none) -> A126441CT-ND
- SW? (x10): footprint (none) -> Footprint_Imports:SW_1571563-4; digikey_part_number CKN10880CT-ND -> 450-2055-1-ND
- SW?: value SW_Push -> SW_RIGHT_ANGLE; footprint (none) -> Footprint_Imports:1825027-8; digikey_part_number CKN10880CT-ND -> 450-1657-ND
- SW?: footprint (none) -> Footprint_Imports:SW_L102021ML04Q; digikey_part_number (none) -> CKC5102-ND
- U? (x2): footprint XDCR_COM-09032 -> Footprint_Imports:XDCR_COM-09032
- U?: digikey_part_number (none) -> 296-47387-1-ND
Connections:
- net +3V3: now also J?.1 (Pin_1), SW?.1, U?.2 (VDD)
- net +5V: now also J?.1 (VBUS), J?.6 (Pin_6)
- net BAT+: now also BT?.+
- net BRIDGE_RX: now also J?.3 (Pin_3), U?.35 (TXD0/IO1)
- net BRIDGE_TX: now also J?.4 (Pin_4), U?.34 (RXD0/IO3)
- net EN: now also U?.3 (EN)
- net GND: now also BT?.-, J?.5 (GND), J?.5 (Pin_5), J?.6 (Shield), U?.1 (GND), U?.15 (GND), U?.38 (GND), U?.39 (GND)
- net I2C_SCL: now also U?.36 (IO22)
- net I2C_SDA: now also U?.33 (IO21)
- net IO0: now also U?.25 (IO0)
- net LEFT_JOY_X: now also U?.13 (IO14)
- net LEFT_JOY_Y: now also U?.16 (IO13)
- net RIGHT_JOY_X: now also U?.9 (IO33)
- net RIGHT_JOY_Y: now also U?.8 (IO32)
- net SW_1: now also U?.27 (IO16)
- net SW_2: now also U?.28 (IO17)
- net SW_3: now also U?.30 (IO18)
- net SW_4: now also U?.31 (IO19)
- net SW_5: now also U?.37 (IO23)
- net SW_6: now also U?.10 (IO25)
- net SW_7: now also U?.11 (IO26)
- net SW_8: now also U?.12 (IO27)
- net TRIG_L: now also SW?.2, U?.7 (IO35)
- net TRIG_R: now also U?.6 (IO34)
- net BRIDGE_DTR: now reaches Q?.2 (E), R?.1, U?.18 (~DTR)
- net BRIDGE_DTR: now also J?.2 (Pin_2)
- net BRIDGE_RTS: now reaches Q?.2 (E), R?.1, U?.19 (~RTS)
- net at U?.8 (USBDP): now also J?.3 (D+)
- net at U?.9 (USBDM): now also J?.2 (D-)
- no-connect marks 29 -> 21
Other:
- note added: "At the time of this design the FT231XQ is difficult to obtain, this \nbackup header will allow for an external programmer to be used if\nthe FT231 cannot be purchased"
- note added: "Backup Programming Header"
- note added: "Battery Holder"
- note added: "Note: This revision utilizes 4 AA batteries for safety and\nsimplicity. Future revisions should look into utilizing lithium \nbased batteries for recharging capability"
- note removed: "Battery Charger"

Commit message: Rough Component layout
Parts:
- removed H?: MountingHole, MountingHole:MountingHole_3.2mm_M3_Pad_Via, symbol Mechanical:MountingHole
- gave numbers to parts that had none: 62
Other:
- moved on the sheet: H1, H2, H3, H4

Commit message: Routed critical signals and power
Parts:
- added C9: 1u, Capacitor_SMD:C_0805_2012Metric_Pad1.18x1.45mm_HandSolder, symbol Device:C
Connections:
- net +3V3: now also C9.1
- net GND: now also C9.2
- net D+: now reaches J1.3 (D+), U2.8 (USBDP)
- net D-: now reaches J1.2 (D-), U2.9 (USBDM)
Changed lines of the file:
@@
 Text Notes 800  7650 0    30   ~ 0
 At the time of this design the FT231XQ is difficult to obtain, this \nbackup header will allow for an external programmer to be used if\nthe FT231 cannot be purchased
+Text Label 1750 5400 0    50   ~ 0
+D-
+Text Label 1750 5500 0    50   ~ 0
+D+
+$Comp
+L Device:C C9
+U 1 1 61B29F1A
+P 2250 4850
+F 0 "C9" H 2365 4896 50  0000 L CNN
+F 1 "1u" H 2365 4805 50  0000 L CNN
+F 2 "Capacitor_SMD:C_0805_2012Metric_Pad1.18x1.45mm_HandSolder" H 2288 4700 50  0001 C CNN
+F 3 "~" H 2250 4850 50  0001 C CNN
+F 4 "1276-1275-1-ND" H 2250 4850 50  0001 C CNN "digikey_part_number"
+	1    2250 4850
+	1    0    0    -1
+$EndComp
+$Comp
+L power:+3.3V #PWR061
+U 1 1 61B2D3A0
+P 2250 4700
+F 0 "#PWR061" H 2250 4550 50  0001 C CNN
+F 1 "+3.3V" H 2265 4873 50  0000 C CNN
+F 2 "" H 2250 4700 50  0001 C CNN
+F 3 "" H 2250 4700 50  0001 C CNN
+	1    2250 4700
+	1    0    0    -1
+$EndComp
+$Comp
+L power:GND #PWR062
+U 1 1 61B2E1BA
+P 2250 5000
+F 0 "#PWR062" H 2250 4750 50  0001 C CNN
+F 1 "GND" H 2255 4827 50  0000 C CNN
+F 2 "" H 2250 5000 50  0001 C CNN
+F 3 "" H 2250 5000 50  0001 C CNN
+	1    2250 5000
+	1    0    0    -1
+$EndComp
 $EndSCHEMATC

Commit message: Completed Routing
Parts:
- added C10, C11: 1u, Capacitor_SMD:C_0805_2012Metric_Pad1.18x1.45mm_HandSolder, symbol Device:C
- SW10, SW11, SW12, SW13, SW2, SW3, SW6, SW7, SW8, SW9: symbol Switch:SW_Push -> Project_Imports:1571563-4
Connections:
- net +3V3: now also C10.1, C11.1
- net EN: now also SW2.3; no longer SW2.2
- net GND: now also C10.2, C11.2
- net IO0: now also SW3.3; no longer SW3.2
- net LEFT_JOY_SW: now also U5.26 (IO4)
- net RIGHT_JOY_SW: now also U5.7 (IO35)
- net RIGHT_JOY_X: now also U5.8 (IO32); no longer U5.9 (IO33)
- net RIGHT_JOY_Y: now also U5.9 (IO33); no longer U5.8 (IO32)
- net SW_1: now also SW6.3, U5.28 (IO17); no longer SW6.2, U5.27 (IO16)
- net SW_2: now also SW7.3, U5.27 (IO16); no longer SW7.2, U5.28 (IO17)
- net SW_3: now also SW8.3, U5.31 (IO19); no longer SW8.2, U5.30 (IO18)
- net SW_4: now also SW9.3, U5.30 (IO18); no longer SW9.2, U5.31 (IO19)
- net SW_5: now also SW10.3, U5.10 (IO25); no longer SW10.2, U5.37 (IO23)
- net SW_6: now also SW11.3, U5.6 (IO34); no longer SW11.2, U5.10 (IO25)
- net SW_7: now also SW12.3, U5.4 (SENSOR_VP); no longer SW12.2, U5.11 (IO26)
- net SW_8: now also SW13.3, U5.11 (IO26); no longer SW13.2, U5.12 (IO27)
- net TRIG_L: now also U5.37 (IO23); no longer U5.7 (IO35)
- net TRIG_R: now also U5.12 (IO27); no longer U5.6 (IO34)
- no-connect marks 21 -> 20
Other:
- moved on the sheet: C6, C7, C8

Commit message: Exported production files for rev 1 to "Revision 1 Production Files"
Parts:
- C10, C11, C3, C5, C8, C9: LCSC_part_number (none) -> C28323
- C2, C4, C7: LCSC_part_number (none) -> C15850
- D2: LCSC_part_number (none) -> C2297
- D3: LCSC_part_number (none) -> C2293
- Q2, Q3: LCSC_part_number (none) -> C20526
- R1, R10, R11, R12, R13, R14, R15, R16, R17, R18, R2, R20, R3, R4, R5, R7, R8, R9: LCSC_part_number (none) -> C17414
- R19, R21: LCSC_part_number (none) -> C17710
- R6: LCSC_part_number (none) -> C17713
- U5: LCSC_part_number (none) -> C473012
Changed lines of the file:
@@
 F 3 "https://www.onsemi.com/pub/Collateral/2N3903-D.PDF" H 5750 5100 50  0001 L CNN
 F 4 "3757-MMBT3904_R1_00001CT-ND" H 5750 5100 50  0001 C CNN "digikey_part_number"
+F 5 "C20526" H 5750 5100 50  0001 C CNN "LCSC_part_number"
 	1    5750 5100
 	1    0    0    -1
@@
 F 3 "https://www.onsemi.com/pub/Collateral/2N3903-D.PDF" H 5750 5700 50  0001 L CNN
 F 4 "3757-MMBT3904_R1_00001CT-ND" H 5750 5700 50  0001 C CNN "digikey_part_number"
+F 5 "C20526" H 5750 5700 50  0001 C CNN "LCSC_part_number"
 	1    5750 5700
 	1    0    0    1
@@
 F 3 "~" H 5350 5700 50  0001 C CNN
 F 4 "RMCF0805JT10K0CT-ND" H 5350 5700 50  0001 C CNN "digikey_part_number"
+F 5 "C17414" H 5350 5700 50  0001 C CNN "LCSC_part_number"
 	1    5350 5700
 	0    -1   -1   0
@@
 F 3 "~" H 5350 5100 50  0001 C CNN
 F 4 "RMCF0805JT10K0CT-ND" H 5350 5100 50  0001 C CNN "digikey_part_number"
+F 5 "C17414" H 5350 5100 50  0001 C CNN "LCSC_part_number"
 	1    5350 5100
 	0    -1   -1   0
@@
 F 3 "~" H 6050 7000 50  0001 C CNN
 F 4 "RMCF0805JT10K0CT-ND" H 6050 7000 50  0001 C CNN "digikey_part_number"
+F 5 "C17414" H 6050 7000 50  0001 C CNN "LCSC_part_number"
 	1    6050 7000
 	1    0    0    -1
@@
 F 3 "~" H 6350 7000 50  0001 C CNN
 F 4 "RMCF0805JT10K0CT-ND" H 6350 7000 50  0001 C CNN "digikey_part_number"
+F 5 "C17414" H 6350 7000 50  0001 C CNN "LCSC_part_number"
 	1    6350 7000
 	1    0    0    -1
@@
 F 3 "~" H 3600 3700 50  0001 C CNN
 F 4 "RMCF0805JT10K0CT-ND" H 3600 3700 50  0001 C CNN "digikey_part_number"
+F 5 "C17414" H 3600 3700 50  0001 C CNN "LCSC_part_number"
 	1    3600 3700
 	1    0    0    -1
@@
 F 3 "~" H 5400 3700 50  0001 C CNN
 F 4 "RMCF0805JT10K0CT-ND" H 5400 3700 50  0001 C CNN "digikey_part_number"
+F 5 "C17414" H 5400 3700 50  0001 C CNN "LCSC_part_number"
 	1    5400 3700
 	1    0    0    -1
@@
 F 3 "~" H 6200 3650 50  0001 C CNN
 F 4 "RMCF0805JT10K0CT-ND" H 6200 3650 50  0001 C CNN "digikey_part_number"
+F 5 "C17414" H 6200 3650 50  0001 C CNN "LCSC_part_number"
 	1    6200 3650
 	1    0    0    -1
@@
 F 3 "~" H 6700 3650 50  0001 C CNN
 F 4 "RMCF0805JT10K0CT-ND" H 6700 3650 50  0001 C CNN "digikey_part_number"
+F 5 "C17414" H 6700 3650 50  0001 C CNN "LCSC_part_number"
 	1    6700 3650
 	1    0    0    -1
@@
 F 3 "~" H 8600 6050 50  0001 C CNN
 F 4 "1276-1275-1-ND" H 8600 6050 50  0001 C CNN "digikey_part_number"
+F 5 "C28323" H 8600 6050 50  0001 C CNN "LCSC_part_number"
 	1    8600 6050
 	1    0    0    -1
@@
 F 3 "~" H 8200 6050 50  0001 C CNN
 F 4 "1276-6455-1-ND" H 8200 6050 50  0001 C CNN "digikey_part_number"
+F 5 "C15850" H 8200 6050 50  0001 C CNN "LCSC_part_number"
 	1    8200 6050
 	1    0    0    -1
@@
 F 3 "~" H 7000 1650 50  0001 C CNN
 F 4 "RMCF0805JT10K0CT-ND" H 7000 1650 50  0001 C CNN "digikey_part_number"
+F 5 "C17414" H 7000 1650 50  0001 C CNN "LCSC_part_number"
 	1    7000 1650
 	1    0    0    -1
@@
 F 3 "~" H 7550 1650 50  0001 C CNN
 F 4 "RMCF0805JT10K0CT-ND" H 7550 1650 50  0001 C CNN "digikey_part_number"
+F 5 "C17414" H 7550 1650 50  0001 C CNN "LCSC_part_number"
 	1    7550 1650
 	1    0    0    -1
@@
 F 3 "~" H 10650 1650 50  0001 C CNN
 F 4 "RMCF0805JT10K0CT-ND" H 10650 1650 50  0001 C CNN "digikey_part_number"
+F 5 "C17414" H 10650 1650 50  0001 C CNN "LCSC_part_number"
 	1    10650 1650
 	1    0    0    -1
@@
 F 3 "~" H 10150 1650 50  0001 C CNN
 F 4 "RMCF0805JT10K0CT-ND" H 10150 1650 50  0001 C CNN "digikey_part_number"
+F 5 "C17414" H 10150 1650 50  0001 C CNN "LCSC_part_number"
 	1    10150 1650
 	1    0    0    -1
@@
 F 3 "~" H 9650 1650 50  0001 C CNN
 F 4 "RMCF0805JT10K0CT-ND" H 9650 1650 50  0001 C CNN "digikey_part_number"
+F 5 "C17414" H 9650 1650 50  0001 C CNN "LCSC_part_number"
 	1    9650 1650
 	1    0    0    -1
@@
 F 3 "~" H 9150 1650 50  0001 C CNN
 F 4 "RMCF0805JT10K0CT-ND" H 9150 1650 50  0001 C CNN "digikey_part_number"
+F 5 "C17414" H 9150 1650 50  0001 C CNN "LCSC_part_number"
 	1    9150 1650
 	1    0    0    -1
@@
 F 3 "~" H 8600 1650 50  0001 C CNN
 F 4 "RMCF0805JT10K0CT-ND" H 8600 1650 50  0001 C CNN "digikey_part_number"
+F 5 "C17414" H 8600 1650 50  0001 C CNN "LCSC_part_number"
 	1    8600 1650
 	1    0    0    -1
@@
 F 3 "~" H 8100 1650 50  0001 C CNN
 F 4 "RMCF0805JT10K0CT-ND" H 8100 1650 50  0001 C CNN "digikey_part_number"
+F 5 "C17414" H 8100 1650 50  0001 C CNN "LCSC_part_number"
 	1    8100 1650
 	1    0    0    -1
@@
 F 3 "~" H 5650 1750 50  0001 C CNN
 F 4 "RMCF0805JT10K0CT-ND" H 5650 1750 50  0001 C CNN "digikey_part_number"
+F 5 "C17414" H 5650 1750 50  0001 C CNN "LCSC_part_number"
 	1    5650 1750
 	1    0    0    -1
@@
 F 3 "~" H 5650 1350 50  0001 C CNN
 F 4 "RMCF0805JT47K0CT-ND" H 5650 1350 50  0001 C CNN "digikey_part_number"
+F 5 "C17713" H 5650 1350 50  0001 C CNN "LCSC_part_number"
 	1    5650 1350
 	1    0    0    -1
@@
 F 3 "~" H 3600 1450 50  0001 C CNN
 F 4 "1276-6455-1-ND" H 3600 1450 50  0001 C CNN "digikey_part_number"
+F 5 "C15850" H 3600 1450 50  0001 C CNN "LCSC_part_number"
 	1    3600 1450
 	1    0    0    -1
@@
 F 3 "~" H 4050 1450 50  0001 C CNN
 F 4 "1276-1275-1-ND" H 4050 1450 50  0001 C CNN "digikey_part_number"
+F 5 "C28323" H 4050 1450 50  0001 C CNN "LCSC_part_number"
 	1    4050 1450
 	1    0    0    -1
@@
 F 3 "~" H 6000 1450 50  0001 C CNN
 F 4 "1276-6455-1-ND" H 6000 1450 50  0001 C CNN "digikey_part_number"
+F 5 "C15850" H 6000 1450 50  0001 C CNN "LCSC_part_number"
 	1    6000 1450
 	1    0    0    -1
@@
 F 3 "~" H 6400 1450 50  0001 C CNN
 F 4 "1276-1275-1-ND" H 6400 1450 50  0001 C CNN "digikey_part_number"
+F 5 "C28323" H 6400 1450 50  0001 C CNN "LCSC_part_number"
 	1    6400 1450
 	1    0    0    -1
@@
 F 3 "~" H 1250 1800 50  0001 C CNN
 F 4 "RMCF0805JT10K0CT-ND" H 1250 1800 50  0001 C CNN "digikey_part_number"
+F 5 "C17414" H 1250 1800 50  0001 C CNN "LCSC_part_number"
 	1    1250 1800
 	1    0    0    -1
@@
 F 3 "~" H 10200 5150 50  0001 C CNN
 F 4 "160-1218-1-ND" H 10200 5150 50  0001 C CNN "digikey_part_number"
+F 5 "C2297" H 10200 5150 50  0001 C CNN "LCSC_part_number"
 	1    10200 5150
 	0    -1   -1   0
@@
 F 3 "~" H 10700 5150 50  0001 C CNN
 F 4 "732-4982-1-ND" H 10700 5150 50  0001 C CNN "digikey_part_number"
+F 5 "C2293" H 10700 5150 50  0001 C CNN "LCSC_part_number"
 	1    10700 5150
 	0    -1   -1   0
@@
 F 3 "~" H 10200 4750 50  0001 C CNN
 F 4 "A126441CT-ND" H 10200 4750 50  0001 C CNN "digikey_part_number"
+F 5 "C17710" H 10200 4750 50  0001 C CNN "LCSC_part_number"
 	1    10200 4750
 	1    0    0    -1
@@
 F 3 "~" H 10700 4750 50  0001 C CNN
 F 4 "A126441CT-ND" H 10700 4750 50  0001 C CNN "digikey_part_number"
+F 5 "C17710" H 10700 4750 50  0001 C CNN "LCSC_part_number"
 	1    10700 4750
 	1    0    0    -1
@@
 F 3 "https://www.espressif.com/sites/default/files/documentation/esp32-wroom-32d_esp32-wroom-32u_datasheet_en.pdf" H 8150 4000 50  0001 C CNN
 F 4 "1965-ESP32-WROOM-32D(4MB)CT-ND" H 8450 3950 50  0001 C CNN "digikey_part_number"
+F 5 "C473012" H 8450 3950 50  0001 C CNN "LCSC_part_number"
 	1    8450 3950
 	1    0    0    -1
@@
 F 3 "~" H 2250 4850 50  0001 C CNN
 F 4 "1276-1275-1-ND" H 2250 4850 50  0001 C CNN "digikey_part_number"
+F 5 "C28323" H 2250 4850 50  0001 C CNN "LCSC_part_number"
 	1    2250 4850
 	1    0    0    -1
@@
 F 3 "~" H 8950 6050 50  0001 C CNN
 F 4 "1276-1275-1-ND" H 8950 6050 50  0001 C CNN "digikey_part_number"
+F 5 "C28323" H 8950 6050 50  0001 C CNN "LCSC_part_number"
 	1    8950 6050
 	1    0    0    -1
@@
 F 3 "~" H 9300 6050 50  0001 C CNN
 F 4 "1276-1275-1-ND" H 9300 6050 50  0001 C CNN "digikey_part_number"
+F 5 "C28323" H 9300 6050 50  0001 C CNN "LCSC_part_number"
 	1    9300 6050
 	1    0    0    -1

Commit message: TODO for revision 2 notes
Other:
- note added: "REVISION 2 TODO: \n - Move left joystick to ADC1 so it can operate with WIFI \n - Switch Buck Converter (Out of stock everywhere)\n - Lithium Ion Battery!"
Changed lines of the file:
@@
 	1    0    0    -1
 $EndComp
+Text Notes 11750 1550 0    98   ~ 0
+REVISION 2 TODO: \n   - Move left joystick to ADC1 so it can operate with WIFI \n   - Switch Buck Converter (Out of stock everywhere)\n   - Lithium Ion Battery!
 $EndSCHEMATC
