File: Makers-Unified-Controller/Makers-Unified-Controller.kicad_pcb (KiCad board)
At the start: 2 copper layers, 130.8 x 76.8 mm, 68 parts, among them J1 USB_B_Micro, J2 backup_PROG, J3 BAT Connector, Q1 PJA3401A_R1_00001, Q2 MMBT3904, Q3 MMBT3904, SW1 SW_DPDT_x2, SW10 SW_Push, SW11 SW_Push, SW12 SW_Push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

Commit message: minor edits to schematic and Ibom
Parts:
- R19, R21: value 470 -> 2.2k
- U3: value MCP73832-2-OT -> MCP73832-2-0T
