File: Makers-Unified-Controller/power_management.kicad_sch (KiCad schematic)
At the start: 16 parts

Commit message: Started PCB - removed unused components from revision 1
Parts:
- gave numbers to parts that had none: 16
Connections:
- no-connect marks 3 -> 1
Changed lines of the file:
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@@
   (junction (at 63.5 46.99) (diameter 0) (color 0 0 0 0)
   )
-  (no_connect (at 50.8 132.08))
-  (no_connect (at 50.8 147.32))
   (no_connect (at 97.79 49.53))
   (wire (pts (xy 210.82 44.45) (xy 214.63 44.45))
@@
   (symbol (lib_id "Device:C") (at 132.08 52.07 0) (unit 1)
     (in_bom yes) (on_board yes)
-    (property "Reference" "C?" (id 0) (at 135.001 50.9016 0)
+    (property "Reference" "C2" (id 0) (at 135.001 50.9016 0)
       (effects (font (size 1.27 1.27)) (justify left))
     )
@@
   (symbol (lib_id "power:GND") (at 57.15 102.87 0) (unit 1)
     (in_bom yes) (on_board yes) (fields_autoplaced)
-    (property "Reference" "#PWR?" (id 0) (at 57.15 109.22 0)
+    (property "Reference" "#PWR0116" (id 0) (at 57.15 109.22 0)
       (effects (font (size 1.27 1.27)) hide)
     )
@@
   (symbol (lib_id "power:GND") (at 152.4 56.388 0) (unit 1)
     (in_bom yes) (on_board yes) (fields_autoplaced)
-    (property "Reference" "#PWR?" (id 0) (at 152.4 62.738 0)
+    (property "Reference" "#PWR0109" (id 0) (at 152.4 62.738 0)
       (effects (font (size 1.27 1.27)) hide)
     )
@@
   (symbol (lib_id "power:GND") (at 132.08 56.388 0) (unit 1)
     (in_bom yes) (on_board yes) (fields_autoplaced)
-    (property "Reference" "#PWR?" (id 0) (at 132.08 62.738 0)
+    (property "Reference" "#PWR0111" (id 0) (at 132.08 62.738 0)
       (effects (font (size 1.27 1.27)) hide)
     )
@@
   (symbol (lib_id "power:GND") (at 63.5 58.42 0) (unit 1)
     (in_bom yes) (on_board yes)
-    (property "Reference" "#PWR?" (id 0) (at 63.5 64.77 0)
+    (property "Reference" "#PWR0107" (id 0) (at 63.5 64.77 0)
       (effects (font (size 1.27 1.27)) hide)
     )
@@
   (symbol (lib_id "Device:D_Schottky") (at 69.85 46.99 180) (unit 1)
     (in_bom yes) (on_board yes)
-    (property "Reference" "D?" (id 0) (at 69.85 41.4782 0))
+    (property "Reference" "D1" (id 0) (at 69.85 41.4782 0))
     (property "Value" "" (id 1) (at 69.85 43.7896 0))
     (property "Footprint" "" (id 2) (at 69.85 46.99 0)
@@
   (symbol (lib_id "power:GND") (at 231.14 57.15 0) (unit 1)
     (in_bom yes) (on_board yes)
-    (property "Reference" "#PWR?" (id 0) (at 231.14 63.5 0)
+    (property "Reference" "#PWR0115" (id 0) (at 231.14 63.5 0)
       (effects (font (size 1.27 1.27)) hide)
     )
@@
   (symbol (lib_id "Device:R") (at 63.5 53.34 0) (unit 1)
     (in_bom yes) (on_board yes)
-    (property "Reference" "R?" (id 0) (at 65.278 52.1716 0)
+    (property "Reference" "R6" (id 0) (at 65.278 52.1716 0)
       (effects (font (size 1.27 1.27)) (justify left))
     )
@@
   (symbol (lib_id "Device:C") (at 231.14 52.07 0) (unit 1)
     (in_bom yes) (on_board yes)
-    (property "Reference" "C?" (id 0) (at 234.061 50.9016 0)
+    (property "Reference" "C12" (id 0) (at 234.061 50.9016 0)
       (effects (font (size 1.27 1.27)) (justify left))
     )
@@
   (symbol (lib_id "Device:C") (at 152.4 52.07 0) (unit 1)
     (in_bom yes) (on_board yes)
-    (property "Reference" "C?" (id 0) (at 155.321 50.9016 0)
+    (property "Reference" "C4" (id 0) (at 155.321 50.9016 0)
       (effects (font (size 1.27 1.27)) (justify left))
     )
@@
   (symbol (lib_id "Device:C") (at 220.98 52.07 0) (unit 1)
     (in_bom yes) (on_board yes)
-    (property "Reference" "C?" (id 0) (at 223.901 50.9016 0)
+    (property "Reference" "C5" (id 0) (at 223.901 50.9016 0)
       (effects (font (size 1.27 1.27)) (justify left))
     )
@@
   (symbol (lib_id "Device:C") (at 241.3 52.07 0) (unit 1)
     (in_bom yes) (on_board yes)
-    (property "Reference" "C?" (id 0) (at 244.221 50.9016 0)
+    (property "Reference" "C13" (id 0) (at 244.221 50.9016 0)
       (effects (font (size 1.27 1.27)) (justify left))
     )
@@
   (symbol (lib_id "Battery_Management:MCP73832-2-OT") (at 57.15 92.71 0) (unit 1)
     (in_bom yes) (on_board yes) (fields_autoplaced)
-    (property "Reference" "U?" (id 0) (at 59.1694 82.55 0)
+    (property "Reference" "U3" (id 0) (at 59.1694 82.55 0)
       (effects (font (size 1.27 1.27)) (justify left))
     )
@@
   (symbol (lib_id "Connector:Conn_01x02_Female") (at 82.55 134.62 0) (mirror y) (unit 1)
     (in_bom yes) (on_board yes) (fields_autoplaced)
-    (property "Reference" "J?" (id 0) (at 83.185 128.778 0))
+    (property "Reference" "J3" (id 0) (at 83.185 128.778 0))
     (property "Value" "" (id 1) (at 83.185 131.318 0))
     (property "Footprint" "" (id 2) (at 82.55 134.62 0)
@@
   (symbol (lib_id "power:GND") (at 93.98 142.24 0) (unit 1)
     (in_bom yes) (on_board yes)
-    (property "Reference" "#PWR?" (id 0) (at 93.98 148.59 0)
+    (property "Reference" "#PWR0118" (id 0) (at 93.98 148.59 0)
       (effects (font (size 1.27 1.27)) hide)
     )
@@
   (symbol (lib_id "Device:C") (at 142.24 52.07 0) (unit 1)
     (in_bom yes) (on_board yes)
-    (property "Reference" "C?" (id 0) (at 145.161 50.9016 0)
+    (property "Reference" "C3" (id 0) (at 145.161 50.9016 0)
       (effects (font (size 1.27 1.27)) (justify left))
     )
@@
   )
   (symbol (lib_id "Project_Imports:PRT-18286") (at 50.8 139.7 270) (unit 1)
-    (in_bom yes) (on_board yes) (fields_autoplaced)
-    (property "Reference" "BT?" (id 0) (at 54.61 137.1345 90)
-      (effects (font (size 1.27 1.27)) (justify left))
-    )
-    (property "Value" "" (id 1) (at 54.61 139.6745 90)
-      (effects (font (size 1.27 1.27)) (justify left))
-    )
-    (property "Footprint" "" (id 2) (at 50.8 139.7 0)
+    (in_bom yes) (on_board yes)
+    (property "Reference" "BT1" (id 0) (at 55.245 131.445 90)
+      (effects (font (size 1.27 1.27)) (justify left))
+    )
+    (property "Value" "" (id 1) (at 59.055 141.605 90)
+      (effects (font (size 1.27 1.27)) (justify left))
+    )
+    (property "Footprint" "" (id 2) (at 62.23 118.11 0)
       (effects (font (size 1.27 1.27)) (justify left bottom) hide)
     )
-    (property "Datasheet" "https://cdn.sparkfun.com/assets/e/3/3/2/7/-KPL623450-1300mAh-3.7V_______________2021-01-21.pdf" (id 3) (at 50.8 139.7 0)
+    (property "Datasheet" "https://cdn.sparkfun.com/assets/e/3/3/2/7/-KPL623450-1300mAh-3.7V_______________2021-01-21.pdf" (id 3) (at 58.42 119.38 0)
       (effects (font (size 1.27 1.27)) (justify left bottom) hide)
     )
-    (property "digikey_part_number" "1568-PRT-18286-ND" (id 4) (at 54.61 142.2145 90)
+    (property "digikey_part_number" "1568-PRT-18286-ND" (id 4) (at 57.785 139.065 90)
       (effects (font (size 0.8382 0.8382)) (justify left))
     )
-    (pin "+")
-    (pin "-")
   )
   (symbol (lib_id "Device:R") (at 44.45 101.6 0) (unit 1)
     (in_bom yes) (on_board yes) (fields_autoplaced)
-    (property "Reference" "R?" (id 0) (at 46.99 100.3299 0)
+    (property "Reference" "R1" (id 0) (at 46.99 100.3299 0)
       (effects (font (size 1.27 1.27)) (justify left))
     )
@@
   (symbol (lib_id "power:GND") (at 142.24 56.388 0) (unit 1)
     (in_bom yes) (on_board yes) (fields_autoplaced)
-    (property "Reference" "#PWR?" (id 0) (at 142.24 62.738 0)
+    (property "Reference" "#PWR0110" (id 0) (at 142.24 62.738 0)
       (effects (font (size 1.27 1.27)) hide)
     )
@@
   (symbol (lib_id "power:GND") (at 220.98 57.15 0) (unit 1)
     (in_bom yes) (on_board yes) (fields_autoplaced)
-    (property "Reference" "#PWR?" (id 0) (at 220.98 63.5 0)
+    (property "Reference" "#PWR0113" (id 0) (at 220.98 63.5 0)
       (effects (font (size 1.27 1.27)) hide)
     )
@@
   (symbol (lib_id "Transistor_FET:FDN340P") (at 77.47 38.1 0) (unit 1)
     (in_bom yes) (on_board yes)
-    (property "Reference" "Q?" (id 0) (at 82.6516 36.9316 0)
+    (property "Reference" "Q1" (id 0) (at 82.6516 36.9316 0)
       (effects (font (size 1.27 1.27)) (justify left))
     )
@@
   (symbol (lib_id "power:GND") (at 181.61 66.802 0) (unit 1)
     (in_bom yes) (on_board yes)
-    (property "Reference" "#PWR?" (id 0) (at 181.61 73.152 0)
+    (property "Reference" "#PWR0112" (id 0) (at 181.61 73.152 0)
       (effects (font (size 1.27 1.27)) hide)
     )
@@
   (symbol (lib_id "power:GND") (at 241.3 57.15 0) (unit 1)
     (in_bom yes) (on_board yes)
-    (property "Reference" "#PWR?" (id 0) (at 241.3 63.5 0)
+    (property "Reference" "#PWR0114" (id 0) (at 241.3 63.5 0)
       (effects (font (size 1.27 1.27)) hide)
     )
@@
   (symbol (lib_id "power:GND") (at 167.64 58.42 0) (unit 1)
     (in_bom yes) (on_board yes)
-    (property "Reference" "#PWR?" (id 0) (at 167.64 64.77 0)
+    (property "Reference" "#PWR0108" (id 0) (at 167.64 64.77 0)
       (effects (font (size 1.27 1.27)) hide)
     )
@@
   (symbol (lib_id "power:GND") (at 44.45 107.95 0) (unit 1)
     (in_bom yes) (on_board yes)
-    (property "Reference" "#PWR?" (id 0) (at 44.45 114.3 0)
+    (property "Reference" "#PWR0117" (id 0) (at 44.45 114.3 0)
       (effects (font (size 1.27 1.27)) hide)
     )
@@
   (symbol (lib_id "Switch:SW_DPDT_x2") (at 92.71 46.99 0) (unit 1)
     (in_bom yes) (on_board yes)
-    (property "Reference" "SW?" (id 0) (at 92.71 39.751 0))
+    (property "Reference" "SW1" (id 0) (at 92.71 39.751 0))
     (property "Value" "" (id 1) (at 92.71 42.0624 0))
     (property "Footprint" "" (id 2) (at 92.71 46.99 0)
@@
   (symbol (lib_id "Device:L") (at 207.01 44.45 90) (unit 1)
     (in_bom yes) (on_board yes) (fields_autoplaced)
-    (property "Reference" "L?" (id 0) (at 207.01 38.1 90))
+    (property "Reference" "L1" (id 0) (at 207.01 38.1 90))
     (property "Value" "" (id 1) (at 207.01 40.64 90))
     (property "Footprint" "" (id 2) (at 207.01 44.45 0)
@@
   (symbol (lib_id "Project_Imports:TPS62046DRCR") (at 181.61 50.8 0) (unit 1)
     (in_bom yes) (on_board yes) (fields_autoplaced)
-    (property "Reference" "U?" (id 0) (at 181.61 33.02 0))
+    (property "Reference" "U6" (id 0) (at 181.61 33.02 0))
     (property "Value" "" (id 1) (at 181.61 35.56 0))
     (property "Footprint" "" (id 2) (at 146.05 22.86 0)

Commit message: fixed BOM item in schematic
Parts:
- BT1: value (none) -> PRT-18286
- C12, C2, C3, C5: value (none) -> 10u
- C13, C4: value (none) -> 1u
- D1: value (none) -> CDBA340-G
- J3: value (none) -> BAT Connector
- L1: value (none) -> 6.2u
- Q1: value (none) -> PJA3401A_R1_00001
- R1: value (none) -> 2.2k
- R6: value (none) -> 10k
- SW1: value (none) -> SW_DPDT_x2
- U3: value (none) -> MCP73832-2-OT
- U6: value (none) -> TPS62046DRCR
Changed lines of the file:
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@@
       (effects (font (size 1.27 1.27)) (justify left))
     )
-    (property "Value" "" (id 1) (at 135.001 53.213 0)
+    (property "Value" "10u" (id 1) (at 135.001 53.213 0)
       (effects (font (size 1.27 1.27)) (justify left))
     )
@@
       (effects (font (size 1.27 1.27)) hide)
     )
-    (property "Value" "" (id 1) (at 57.15 107.95 0))
+    (property "Value" "GND" (id 1) (at 57.15 107.95 0))
     (property "Footprint" "" (id 2) (at 57.15 102.87 0)
       (effects (font (size 1.27 1.27)) hide)
@@
     (in_bom yes) (on_board yes)
     (property "Reference" "D1" (id 0) (at 69.85 41.4782 0))
-    (property "Value" "" (id 1) (at 69.85 43.7896 0))
+    (property "Value" "CDBA340-G" (id 1) (at 69.85 43.7896 0))
     (property "Footprint" "" (id 2) (at 69.85 46.99 0)
       (effects (font (size 1.27 1.27)) hide)
@@
       (effects (font (size 1.27 1.27)) (justify left))
     )
-    (property "Value" "" (id 1) (at 65.278 54.483 0)
+    (property "Value" "10k" (id 1) (at 65.278 54.483 0)
       (effects (font (size 1.27 1.27)) (justify left))
     )
@@
       (effects (font (size 1.27 1.27)) (justify left))
     )
-    (property "Value" "" (id 1) (at 234.061 53.213 0)
+    (property "Value" "10u" (id 1) (at 234.061 53.213 0)
       (effects (font (size 1.27 1.27)) (justify left))
     )
@@
       (effects (font (size 1.27 1.27)) (justify left))
     )
-    (property "Value" "" (id 1) (at 155.321 53.213 0)
+    (property "Value" "1u" (id 1) (at 155.321 53.213 0)
       (effects (font (size 1.27 1.27)) (justify left))
     )
@@
       (effects (font (size 1.27 1.27)) (justify left))
     )
-    (property "Value" "" (id 1) (at 223.901 53.213 0)
+    (property "Value" "10u" (id 1) (at 223.901 53.213 0)
       (effects (font (size 1.27 1.27)) (justify left))
     )
@@
       (effects (font (size 1.27 1.27)) (justify left))
     )
-    (property "Value" "" (id 1) (at 244.221 53.213 0)
+    (property "Value" "1u" (id 1) (at 244.221 53.213 0)
       (effects (font (size 1.27 1.27)) (justify left))
     )
@@
       (effects (font (size 1.27 1.27)) (justify left))
     )
-    (property "Value" "" (id 1) (at 59.1694 85.09 0)
+    (property "Value" "MCP73832-2-OT" (id 1) (at 59.1694 85.09 0)
       (effects (font (size 1.27 1.27)) (justify left))
     )
@@
     (in_bom yes) (on_board yes) (fields_autoplaced)
     (property "Reference" "J3" (id 0) (at 83.185 128.778 0))
-    (property "Value" "" (id 1) (at 83.185 131.318 0))
+    (property "Value" "BAT Connector" (id 1) (at 83.185 131.318 0))
     (property "Footprint" "" (id 2) (at 82.55 134.62 0)
       (effects (font (size 1.27 1.27)) hide)
@@
       (effects (font (size 1.27 1.27)) (justify left))
     )
-    (property "Value" "" (id 1) (at 145.161 53.213 0)
+    (property "Value" "10u" (id 1) (at 145.161 53.213 0)
       (effects (font (size 1.27 1.27)) (justify left))
     )
@@
       (effects (font (size 1.27 1.27)) (justify left))
     )
-    (property "Value" "" (id 1) (at 59.055 141.605 90)
+    (property "Value" "PRT-18286" (id 1) (at 59.055 141.605 90)
       (effects (font (size 1.27 1.27)) (justify left))
     )
@@
       (effects (font (size 1.27 1.27)) (justify left))
     )
-    (property "Value" "" (id 1) (at 46.99 102.8699 0)
+    (property "Value" "2.2k" (id 1) (at 46.99 102.8699 0)
       (effects (font (size 1.27 1.27)) (justify left))
     )
@@
       (effects (font (size 1.27 1.27)) (justify left))
     )
-    (property "Value" "" (id 1) (at 82.55 34.29 0)
+    (property "Value" "PJA3401A_R1_00001" (id 1) (at 82.55 34.29 0)
       (effects (font (size 1.27 1.27)) (justify left))
     )
@@
       (effects (font (size 1.27 1.27)) hide)
     )
-    (property "Value" "" (id 1) (at 44.45 111.76 0))
+    (property "Value" "GND" (id 1) (at 44.45 111.76 0))
     (property "Footprint" "" (id 2) (at 44.45 107.95 0)
       (effects (font (size 1.27 1.27)) hide)
@@
     (in_bom yes) (on_board yes)
     (property "Reference" "SW1" (id 0) (at 92.71 39.751 0))
-    (property "Value" "" (id 1) (at 92.71 42.0624 0))
+    (property "Value" "SW_DPDT_x2" (id 1) (at 92.71 42.0624 0))
     (property "Footprint" "" (id 2) (at 92.71 46.99 0)
       (effects (font (size 1.27 1.27)) hide)
@@
     (in_bom yes) (on_board yes) (fields_autoplaced)
     (property "Reference" "L1" (id 0) (at 207.01 38.1 90))
-    (property "Value" "" (id 1) (at 207.01 40.64 90))
+    (property "Value" "6.2u" (id 1) (at 207.01 40.64 90))
     (property "Footprint" "" (id 2) (at 207.01 44.45 0)
       (effects (font (size 1.27 1.27)) hide)
@@
     (in_bom yes) (on_board yes) (fields_autoplaced)
     (property "Reference" "U6" (id 0) (at 181.61 33.02 0))
-    (property "Value" "" (id 1) (at 181.61 35.56 0))
+    (property "Value" "TPS62046DRCR" (id 1) (at 181.61 35.56 0))
     (property "Footprint" "" (id 2) (at 146.05 22.86 0)
       (effects (font (size 1.27 1.27)) hide)

Commit message: Completed routing - TODO final checks
Parts:
- BT1: value PRT-18286 -> (none)
- C12, C2, C3, C5: value 10u -> (none)
- C13, C4: value 1u -> (none)
- D1: value CDBA340-G -> (none)
- J3: value BAT Connector -> (none)
- L1: value 6.2u -> (none)
- Q1: value PJA3401A_R1_00001 -> (none)
- R1: value 2.2k -> (none)
- R6: value 10k -> (none)
- SW1: value SW_DPDT_x2 -> (none)
- U3: value MCP73832-2-OT -> (none)
- U6: value TPS62046DRCR -> (none); digikey (none) -> 296-15902-1-ND
Connections:
- net GND: now also U6.11 (PAD)
- net BUCK_SW: now reaches L1.1, U6.7 (SW), U6.8 (SW)

Commit message: Finalized layout and exported files
Parts:
- BT1: footprint (none) -> Footprint_Imports:PRT18286
- Q1: footprint (none) -> Package_TO_SOT_SMD:SOT-23
- U3: footprint (none) -> Package_TO_SOT_SMD:SOT-23-5
- U6: footprint (none) -> Package_SON:VSON-10-1EP_3x3mm_P0.5mm_EP1.2x2mm_ThermalVias
Other:
- note added: "Connector for battery used is a JST-XH footprint was modified to include +/- symbols on PCB"
- note added: "MCP73832 supplies USB charging capabilities for the lithium battery. (Technically this doesn't need to be populated)"
- note added: "Note, this is just a standin for the battery, power flows into the JST connector. The only reason this is here is to include a footprint on the PCB and a BOM item in the .csv parts list"
- note added: "Power Management - This sub-system handles the generation of 3.3V for the greater system from either USB or the lithium ion battery."
- note removed: "Note, this is just a standin for the battery, power flows into the JST connector"
- company: (none) -> Makers @ Oakland University
- title: (none) -> Makers Unified Controller
- moved on the sheet: BT1, C12, C13, C2, C3, C4, C5, D1, J3, L1, Q1, R6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

Commit message: minor edits
Parts:
- BT1: value (none) -> PRT-18286; footprint Footprint_Imports:PRT18286 -> (none)
- C12, C2, C3, C5: value (none) -> 10u
- C13, C4: value (none) -> 1u
- D1: value (none) -> CDBA340-G
- J3: value (none) -> BAT Connector
- L1: value (none) -> 6.2u
- Q1: value (none) -> PJA3401A_R1_00001; footprint Package_TO_SOT_SMD:SOT-23 -> (none)
- R1: value (none) -> 2.2k
- R6: value (none) -> 10k
- SW1: value (none) -> SW_DPDT_x2
- U3: footprint Package_TO_SOT_SMD:SOT-23-5 -> (none)
- U6: value (none) -> TPS62046DRCR; footprint Package_SON:VSON-10-1EP_3x3mm_P0.5mm_EP1.2x2mm_ThermalVias -> (none)
Changed lines of the file:
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@@
       (effects (font (size 1.27 1.27)) (justify left))
     )
-    (property "Value" "" (id 1) (at 135.001 46.228 0)
+    (property "Value" "10u" (id 1) (at 135.001 46.228 0)
       (effects (font (size 1.27 1.27)) (justify left))
     )
@@
     (in_bom yes) (on_board yes)
     (property "Reference" "D1" (id 0) (at 69.85 34.4932 0))
-    (property "Value" "" (id 1) (at 69.85 36.8046 0))
+    (property "Value" "CDBA340-G" (id 1) (at 69.85 36.8046 0))
     (property "Footprint" "" (id 2) (at 69.85 40.005 0)
       (effects (font (size 1.27 1.27)) hide)
@@
       (effects (font (size 1.27 1.27)) (justify left))
     )
-    (property "Value" "" (id 1) (at 65.278 47.498 0)
+    (property "Value" "10k" (id 1) (at 65.278 47.498 0)
       (effects (font (size 1.27 1.27)) (justify left))
     )
@@
       (effects (font (size 1.27 1.27)) (justify left))
     )
-    (property "Value" "" (id 1) (at 234.061 46.228 0)
+    (property "Value" "10u" (id 1) (at 234.061 46.228 0)
       (effects (font (size 1.27 1.27)) (justify left))
     )
@@
       (effects (font (size 1.27 1.27)) (justify left))
     )
-    (property "Value" "" (id 1) (at 155.321 46.228 0)
+    (property "Value" "1u" (id 1) (at 155.321 46.228 0)
       (effects (font (size 1.27 1.27)) (justify left))
     )
@@
       (effects (font (size 1.27 1.27)) (justify left))
     )
-    (property "Value" "" (id 1) (at 223.901 46.228 0)
+    (property "Value" "10u" (id 1) (at 223.901 46.228 0)
       (effects (font (size 1.27 1.27)) (justify left))
     )
@@
       (effects (font (size 1.27 1.27)) (justify left))
     )
-    (property "Value" "" (id 1) (at 244.221 46.228 0)
+    (property "Value" "1u" (id 1) (at 244.221 46.228 0)
       (effects (font (size 1.27 1.27)) (justify left))
     )
@@
       (effects (font (size 1.27 1.27)) (justify left))
     )
-    (property "Footprint" "Package_TO_SOT_SMD:SOT-23-5" (id 2) (at 58.42 99.06 0)
+    (property "Footprint" "" (id 2) (at 58.42 99.06 0)
       (effects (font (size 1.27 1.27) italic) (justify left) hide)
     )
@@
     (in_bom yes) (on_board yes) (fields_autoplaced)
     (property "Reference" "J3" (id 0) (at 81.915 133.858 0))
-    (property "Value" "" (id 1) (at 81.915 136.398 0))
+    (property "Value" "BAT Connector" (id 1) (at 81.915 136.398 0))
     (property "Footprint" "" (id 2) (at 81.28 139.7 0)
       (effects (font (size 1.27 1.27)) hide)
@@
       (effects (font (size 1.27 1.27)) (justify left))
     )
-    (property "Value" "" (id 1) (at 145.161 46.228 0)
+    (property "Value" "10u" (id 1) (at 145.161 46.228 0)
       (effects (font (size 1.27 1.27)) (justify left))
     )
@@
       (effects (font (size 1.27 1.27)) (justify left))
     )
-    (property "Value" "" (id 1) (at 57.785 146.685 90)
-      (effects (font (size 1.27 1.27)) (justify left))
-    )
-    (property "Footprint" "Footprint_Imports:PRT18286" (id 2) (at 60.96 123.19 0)
+    (property "Value" "PRT-18286" (id 1) (at 57.785 146.685 90)
+      (effects (font (size 1.27 1.27)) (justify left))
+    )
+    (property "Footprint" "" (id 2) (at 60.96 123.19 0)
       (effects (font (size 1.27 1.27)) (justify left bottom) hide)
     )
@@
       (effects (font (size 1.27 1.27)) (justify left))
     )
-    (property "Value" "" (id 1) (at 46.99 102.8699 0)
+    (property "Value" "2.2k" (id 1) (at 46.99 102.8699 0)
       (effects (font (size 1.27 1.27)) (justify left))
     )
@@
       (effects (font (size 1.27 1.27)) (justify left))
     )
-    (property "Value" "" (id 1) (at 82.55 27.305 0)
-      (effects (font (size 1.27 1.27)) (justify left))
-    )
-    (property "Footprint" "Package_TO_SOT_SMD:SOT-23" (id 2) (at 82.55 33.02 0)
+    (property "Value" "PJA3401A_R1_00001" (id 1) (at 82.55 27.305 0)
+      (effects (font (size 1.27 1.27)) (justify left))
+    )
+    (property "Footprint" "" (id 2) (at 82.55 33.02 0)
       (effects (font (size 1.27 1.27) italic) (justify left) hide)
     )
@@
     (in_bom yes) (on_board yes)
     (property "Reference" "SW1" (id 0) (at 92.71 32.766 0))
-    (property "Value" "" (id 1) (at 92.71 35.0774 0))
+    (property "Value" "SW_DPDT_x2" (id 1) (at 92.71 35.0774 0))
     (property "Footprint" "" (id 2) (at 92.71 40.005 0)
       (effects (font (size 1.27 1.27)) hide)
@@
     (in_bom yes) (on_board yes) (fields_autoplaced)
     (property "Reference" "L1" (id 0) (at 207.01 31.115 90))
-    (property "Value" "" (id 1) (at 207.01 33.655 90))
+    (property "Value" "6.2u" (id 1) (at 207.01 33.655 90))
     (property "Footprint" "" (id 2) (at 207.01 37.465 0)
       (effects (font (size 1.27 1.27)) hide)
@@
     (in_bom yes) (on_board yes) (fields_autoplaced)
     (property "Reference" "U6" (id 0) (at 181.61 26.035 0))
-    (property "Value" "" (id 1) (at 181.61 28.575 0))
-    (property "Footprint" "Package_SON:VSON-10-1EP_3x3mm_P0.5mm_EP1.2x2mm_ThermalVias" (id 2) (at 146.05 15.875 0)
-      (effects (font (size 1.27 1.27)) hide)
-    )
+    (property "Value" "TPS62046DRCR" (id 1) (at 181.61 28.575 0))
+    (property "Footprint" "" (id 2) (at 146.05 15.875 0)
+      (effects (font (size 1.27 1.27)) hide)
+    )
